File: kicad/if_chg_board/if_chg_board.kicad_sch (KiCad schematic)
At the start: 42 parts, among them J1 USB_B_Micro, J2 B2B-ZH, J3 B2B-ZH, J4 Conn_01x05, Q1 SS8050-G, Q2 SS8050-G, SW1 B3U-1000P, SW2 B3U-1000P, U1 AMS1117-3.3, U2 LTC4054ES5-4.2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

Commit message: Update if_chg_board
Signed-off-by: Kazuki Iida <elkel53930@gmail.com>
Parts:
- added H1, H2, H3, H4: Φ3.2 M3, MountingHole:MountingHole_3.2mm_M3, symbol Mechanical:MountingHole
- added J5: B2B-ZH, Connector_PinHeader_2.54mm:PinHeader_1x02_P2.54mm_Vertical, symbol Connector_Generic:Conn_01x02
Connections:
- net +5V: now also J5.2 (Pin_2)
- net GND: now also J5.1 (Pin_1)
Changed lines of the file:
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@@
+    (stroke (width 0) (type default))
+  )
+  (wire (pts (xy 109.22 45.72) (xy 109.22 43.18))
     (stroke (width 0) (type default))
   )
@@
     (stroke (width 0) (type default))
   )
+  (wire (pts (xy 109.22 38.1) (xy 109.22 40.64))
+    (stroke (width 0) (type default))
+  )
   (wire (pts (xy 52.705 96.52) (xy 52.705 98.425))
     (stroke (width 0) (type default))
@@
     (stroke (width 0) (type default))
   )
+  (wire (pts (xy 109.22 40.64) (xy 111.76 40.64))
+    (stroke (width 0) (type default))
+  )
   (wire (pts (xy 54.61 45.72) (xy 66.04 45.72))
     (stroke (width 0) (type default))
@@
   )
   (wire (pts (xy 227.965 57.785) (xy 200.025 57.785))
+    (stroke (width 0) (type default))
+  )
+  (wire (pts (xy 109.22 43.18) (xy 111.76 43.18))
     (stroke (width 0) (type default))
   )
@@
     )
   )
+  (symbol (lib_id "Mechanical:MountingHole") (at 152.4 172.72 0) (unit 1)
+    (in_bom yes) (on_board yes) (dnp no)
+    (property "Reference" "H4" (at 154.94 172.085 0)
+      (effects (font (size 1.27 1.27)) (justify left))
+    )
+    (property "Value" "Φ3.2 M3" (at 154.94 174.625 0)
+      (effects (font (size 1.27 1.27)) (justify left))
+    )
+    (property "Footprint" "MountingHole:MountingHole_3.2mm_M3" (at 152.4 172.72 0)
+      (effects (font (size 1.27 1.27)) hide)
+    )
+    (property "Datasheet" "~" (at 152.4 172.72 0)
+      (effects (font (size 1.27 1.27)) hide)
+    )
+    (instances
+      (project "if_chg_board"
+        (path "/442b792c-8cde-473e-a235-3fac6ca0f027"
+          (reference "H4") (unit 1)
+        )
+      )
+    )
+  )
   (symbol (lib_id "power:GND") (at 238.76 148.59 0) (unit 1)
     (in_bom yes) (on_board yes) (dnp no) (fields_autoplaced)
@@
         (path "/442b792c-8cde-473e-a235-3fac6ca0f027"
           (reference "R6") (unit 1)
+        )
+      )
+    )
+  )
+  (symbol (lib_id "Mechanical:MountingHole") (at 152.4 167.64 0) (unit 1)
+    (in_bom yes) (on_board yes) (dnp no)
+    (property "Reference" "H3" (at 154.94 167.005 0)
+      (effects (font (size 1.27 1.27)) (justify left))
+    )
+    (property "Value" "Φ3.2 M3" (at 154.94 169.545 0)
+      (effects (font (size 1.27 1.27)) (justify left))
+    )
+    (property "Footprint" "MountingHole:MountingHole_3.2mm_M3" (at 152.4 167.64 0)
+      (effects (font (size 1.27 1.27)) hide)
+    )
+    (property "Datasheet" "~" (at 152.4 167.64 0)
+      (effects (font (size 1.27 1.27)) hide)
+    )
+    (instances
+      (project "if_chg_board"
+        (path "/442b792c-8cde-473e-a235-3fac6ca0f027"
+          (reference "H3") (unit 1)
         )
       )
@@
     )
   )
+  (symbol (lib_id "Connector_Generic:Conn_01x02") (at 116.84 43.18 0) (mirror x) (unit 1)
+    (in_bom yes) (on_board yes) (dnp no)
+    (property "Reference" "J5" (at 120.015 42.545 0)
+      (effects (font (size 1.27 1.27)) (justify left))
+    )
+    (property "Value" "B2B-ZH" (at 120.015 40.005 0)
+      (effects (font (size 1.27 1.27)) (justify left))
+    )
+    (property "Footprint" "Connector_PinHeader_2.54mm:PinHeader_1x02_P2.54mm_Vertical" (at 116.84 43.18 0)
+      (effects (font (size 1.27 1.27)) hide)
+    )
+    (property "Datasheet" "~" (at 116.84 43.18 0)
+      (effects (font (size 1.27 1.27)) hide)
+    )
+    (pin "1")
+    (pin "2")
+    (instances
+      (project "if_chg_board"
+        (path "/442b792c-8cde-473e-a235-3fac6ca0f027"
+          (reference "J5") (unit 1)
+        )
+      )
+    )
+  )
   (symbol (lib_id "power:+5V") (at 66.04 31.75 0) (unit 1)
     (in_bom yes) (on_board yes) (dnp no) (fields_autoplaced)
@@
         (path "/442b792c-8cde-473e-a235-3fac6ca0f027"
           (reference "D4") (unit 1)
+        )
+      )
+    )
+  )
+  (symbol (lib_id "power:+5V") (at 109.22 38.1 0) (unit 1)
+    (in_bom yes) (on_board yes) (dnp no) (fields_autoplaced)
+    (property "Reference" "#PWR038" (at 109.22 41.91 0)
+      (effects (font (size 1.27 1.27)) hide)
+    )
+    (property "Value" "+5V" (at 109.22 34.29 0)
+      (effects (font (size 1.27 1.27)))
+    )
+    (property "Footprint" "" (at 109.22 38.1 0)
+      (effects (font (size 1.27 1.27)) hide)
+    )
+    (property "Datasheet" "" (at 109.22 38.1 0)
+      (effects (font (size 1.27 1.27)) hide)
+    )
+    (pin "1")
+    (instances
+      (project "if_chg_board"
+        (path "/442b792c-8cde-473e-a235-3fac6ca0f027"
+          (reference "#PWR038") (unit 1)
         )
       )
@@
     )
   )
+  (symbol (lib_id "Mechanical:MountingHole") (at 137.16 167.64 0) (unit 1)
+    (in_bom yes) (on_board yes) (dnp no)
+    (property "Reference" "H1" (at 139.7 167.005 0)
+      (effects (font (size 1.27 1.27)) (justify left))
+    )
+    (property "Value" "Φ3.2 M3" (at 139.7 169.545 0)
+      (effects (font (size 1.27 1.27)) (justify left))
+    )
+    (property "Footprint" "MountingHole:MountingHole_3.2mm_M3" (at 137.16 167.64 0)
+      (effects (font (size 1.27 1.27)) hide)
+    )
+    (property "Datasheet" "~" (at 137.16 167.64 0)
+      (effects (font (size 1.27 1.27)) hide)
+    )
+    (instances
+      (project "if_chg_board"
+        (path "/442b792c-8cde-473e-a235-3fac6ca0f027"
+          (reference "H1") (unit 1)
+        )
+      )
+    )
+  )
   (symbol (lib_id "power:+5V") (at 63.5 114.935 0) (unit 1)
     (in_bom yes) (on_board yes) (dnp no) (fields_autoplaced)
@@
     )
   )
+  (symbol (lib_id "power:GND") (at 109.22 45.72 0) (unit 1)
+    (in_bom yes) (on_board yes) (dnp no) (fields_autoplaced)
+    (property "Reference" "#PWR037" (at 109.22 52.07 0)
+      (effects (font (size 1.27 1.27)) hide)
+    )
+    (property "Value" "GND" (at 109.22 50.8 0)
+      (effects (font (size 1.27 1.27)))
+    )
+    (property "Footprint" "" (at 109.22 45.72 0)
+      (effects (font (size 1.27 1.27)) hide)
+    )
+    (property "Datasheet" "" (at 109.22 45.72 0)
+      (effects (font (size 1.27 1.27)) hide)
+    )
+    (pin "1")
+    (instances
+      (project "if_chg_board"
+        (path "/442b792c-8cde-473e-a235-3fac6ca0f027"
+          (reference "#PWR037") (unit 1)
+        )
+      )
+    )
+  )
   (symbol (lib_id "power:+3.3V") (at 143.51 54.61 0) (unit 1)
     (in_bom yes) (on_board yes) (dnp no) (fields_autoplaced)
@@
         )
       )
+    )
+  )
+  (symbol (lib_id "Mechanical:MountingHole") (at 137.16 172.72 0) (unit 1)
+    (in_bom yes) (on_board yes) (dnp no)
+    (property "Reference" "H2" (at 139.7 172.085 0)
+      (effects (font (size 1.27 1.27)) (justify left))
+    )
+    (property "Value" "Φ3.2 M3" (at 139.7 174.625 0)
+      (effects (font (size 1.27 1.27)) (justify left))
+    )
+    (property "Footprint" "MountingHole:MountingHole_3.2mm_M3" (at 137.16 172.72 0)
+      (effects (font (size 1.27 1.27)) hide)
+    )
+    (property "Datasheet" "~" (at 137.16 172.72 0)
+      (effects (font (size 1.27 1.27)) hide)
+    )
+    (instances
+      (project "if_chg_board"
+        (path "/442b792c-8cde-473e-a235-3fac6ca0f027"
+          (reference "H2") (unit 1)
+        )
+      )

Commit message: Fix battery charge current
Signed-off-by: Kazuki Iida <elkel53930@gmail.com>
Parts:
- R1, R2: value 1608 1.2K -> 1608 12K
Changed lines of the file:
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@@
       (effects (font (size 1.27 1.27)) (justify left))
     )
-    (property "Value" "1608 1.2K" (at 26.67 123.825 0)
+    (property "Value" "1608 12K" (at 26.67 123.825 0)
       (effects (font (size 1.27 1.27)) (justify left))
     )
@@
       (effects (font (size 1.27 1.27)) (justify left))
     )
-    (property "Value" "1608 1.2K" (at 26.67 166.37 0)
-      (effects (font (size 1.27 1.27)) (justify left))
-    )
+    (property "Value" "1608 12K" (at 26.67 166.37 0)
+      (effects (font (size 1.27 1.27)) (justify left))
+    )
