File: kicad/extraice/extraice.kicad_pcb (KiCad board)
At the start: 2 copper layers, 77 x 57.8 mm, 72 parts, among them J1 Conn_01x02, J10 Conn_01x02, J3 EncSide, J4 MainSide, J5 Conn_01x05, J6 EncSide, J7 MainSide, J8 Conn_01x02, J9 Conn_01x02, Q1 L-31ROPT1C, Q2 L-31ROPT1C, Q3 L-31ROPT1C, Q4 L-31ROPT1C, SW1 PCM12SMTR, SW2 B3U-1000P, U1 DG2034EDN, U10 DRV8837C, U11 DRV8837C, U12 AS5047D, U2 BCR421, U3 MUN12AD01-SG, U4 MB85RC64TA, U5 LSM6DSR, U6 XC6221B302GR, U7 ESP32-S3-FN8, U8 AS5047D, U9 DRV8837C, X1 ECS-2520MVLC-400-BN

Commit message: Fix problems identified during implementation
- ESP32 supports only crystal oscillator, not resonator.
- The package and capacitance of capacitor C1 were incorrect.
- Fix a ESP32 pin name. GPIO15 -> GPIO14.

Signed-off-by: Kazuki Iida <elkel53930@gmail.com>
Parts:
- C1: value 3225 25V 22uF -> 1608 35V 1uF
- X1: value ECS-2520MVLC-400-BN -> 830108208709
Connections:
- X1 pad 4: +3V0 -> GND
Routing:
- net +3V0: track 165.3 -> 162.3 mm, vias 16 -> 15
Changed lines of the file:
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@@
         (effects (font (size 0.6 0.6) (thickness 0.1)))
     )
-    (fp_text value "3225 25V 22uF" (at 0 1.43) (layer "F.Fab") hide
+    (fp_text value "1608 35V 1uF" (at 0 1.43) (layer "F.Fab") hide
         (effects (font (size 0.6 0.6) (thickness 0.1)))
     )
@@
     (property "Sheetfile" "extraice.kicad_sch")
     (property "Sheetname" "")
-    (property "ki_description" "HCMOS Crystal Clock Oscillator, 2.5x2.0 mm SMD")
-    (property "ki_keywords" "Crystal Clock Oscillator ECS SMD")
+    (property "ki_description" "Four pin crystal, GND on pins 2 and 4")
+    (property "ki_keywords" "quartz ceramic resonator oscillator")
     (attr smd)
     (fp_text reference "X1" (at -2 0.3) (layer "F.SilkS")
         (effects (font (size 0.6 0.6) (thickness 0.1)))
     )
-    (fp_text value "ECS-2520MVLC-400-BN" (at 0 2.5) (layer "F.Fab") hide
+    (fp_text value "830108208709" (at 0 2.5) (layer "F.Fab") hide
         (effects (font (size 0.6 0.6) (thickness 0.1)))
     )
@@
       (stroke (width 0.1) (type solid)) (layer "F.Fab"))
     (pad "1" smd roundrect (at -0.725 -0.925) (size 0.8 0.9) (layers "F.Cu" "F.Paste" "F.Mask") (roundrect_rratio 0.25)
-      (net 93 "Net-(U7-XTAL_P)") (pinfunction "Tri-State") (pintype "input"))
+      (net 93 "Net-(U7-XTAL_P)") (pinfunction "1") (pintype "passive"))
     (pad "2" smd roundrect (at -0.725 0.925) (size 0.8 0.9) (layers "F.Cu" "F.Paste" "F.Mask") (roundrect_rratio 0.25)
-      (net 1 "GND") (pinfunction "GND") (pintype "power_in"))
+      (net 1 "GND") (pinfunction "2") (pintype "passive"))
     (pad "3" smd roundrect (at 0.725 0.925) (size 0.8 0.9) (layers "F.Cu" "F.Paste" "F.Mask") (roundrect_rratio 0.25)
-      (net 92 "Net-(U7-XTAL_N)") (pinfunction "OUT") (pintype "output"))
+      (net 92 "Net-(U7-XTAL_N)") (pinfunction "3") (pintype "passive"))
     (pad "4" smd roundrect (at 0.725 -0.925) (size 0.8 0.9) (layers "F.Cu" "F.Paste" "F.Mask") (roundrect_rratio 0.25)
-      (net 3 "+3V0") (pinfunction "VDD") (pintype "power_in"))
+      (net 1 "GND") (pinfunction "4") (pintype "passive"))
     (model "${KICAD6_3DMODEL_DIR}/Oscillator.3dshapes/Oscillator_SMD_ECS_2520MV-xxx-xx-4Pin_2.5x2.0mm.wrl"
       (offset (xyz 0 0 0))
@@
       (net 71 "/SPI1_MOSI") (pinfunction "GPIO13") (pintype "bidirectional"))
     (pad "19" smd roundrect (at -1 3.45 270) (size 0.2 0.8) (layers "F.Cu" "F.Paste" "F.Mask") (roundrect_rratio 0.25)
-      (net 68 "/SEN_LED_ENA") (pinfunction "GPIO15") (pintype "bidirectional"))
+      (net 68 "/SEN_LED_ENA") (pinfunction "GPIO14") (pintype "bidirectional"))
     (pad "20" smd roundrect (at -0.6 3.45 270) (size 0.2 0.8) (layers "F.Cu" "F.Paste" "F.Mask") (roundrect_rratio 0.25)
       (net 3 "+3V0") (pinfunction "VDD3P3_RTC") (pintype "power_in"))
@@
   (segment (start 130.5 116.5) (end 129.5 116.5) (width 0.15) (layer "F.Cu") (net 3))
   (segment (start 141.8 115.05) (end 141.8 114.670674) (width 0.15) (layer "F.Cu") (net 3))
-  (segment (start 147.725 115.975) (end 147.3 116.4) (width 0.3) (layer "F.Cu") (net 3))
   (segment (start 143.755124 130.7745) (end 143.896545 130.7745) (width 0.15) (layer "F.Cu") (net 3))
   (segment (start 144 116.3) (end 143.45 116.3) (width 0.15) (layer "F.Cu") (net 3))
@@
   (segment (start 129.395 117.5) (end 129.245 117.35) (width 0.15) (layer "F.Cu") (net 3))
   (segment (start 145.35 124.6) (end 145.35 123.35) (width 0.5) (layer "F.Cu") (net 3))
-  (segment (start 147.3 116.4) (end 147.1 116.4) (width 0.3) (layer "F.Cu") (net 3))
   (segment (start 133.8 117.9) (end 133.22 117.9) (width 0.15) (layer "F.Cu") (net 3))
   (segment (start 129.245 116.755) (end 129.245 117.35) (width 0.15) (layer "F.Cu") (net 3))
@@
   (via (at 145.3 123.3) (size 0.5) (drill 0.3) (layers "F.Cu" "B.Cu") (net 3))
   (via (at 130 99.5) (size 0.5) (drill 0.3) (layers "F.Cu" "B.Cu") (net 3))
-  (via (at 147.1 116.4) (size 0.5) (drill 0.3) (layers "F.Cu" "B.Cu") (net 3))
   (via (at 130.8 120) (size 0.5) (drill 0.3) (layers "F.Cu" "B.Cu") (net 3))
   (via (at 145.3 116.1) (size 0.5) (drill 0.3) (layers "F.Cu" "B.Cu") (net 3))
@@
   (segment (start 145 116.4) (end 145.3 116.1) (width 0.3) (layer "B.Cu") (net 3))
   (segment (start 136.788966 84.815634) (end 135.649053 85.955547) (width 0.2) (layer "B.Cu") (net 3))
-  (segment (start 145 116.8) (end 146.7 116.8) (width 0.3) (layer "B.Cu") (net 3))
   (segment (start 145.3 115.6) (end 144.5 114.8) (width 0.3) (layer "B.Cu") (net 3))
   (segment (start 145.3 116.1) (end 145.3 115.6) (width 0.3) (layer "B.Cu") (net 3))
@@
   (segment (start 145.3 123.3) (end 144.9 123.7) (width 0.3) (layer "B.Cu") (net 3))
   (segment (start 130.8 118.1) (end 131.4 117.5) (width 0.15) (layer "B.Cu") (net 3))
-  (segment (start 146.7 116.8) (end 147.1 116.4) (width 0.3) (layer "B.Cu") (net 3))
   (segment (start 144.80659 85.00659) (end 144.80659 84.815634) (width 0.2) (layer "B.Cu") (net 3))
   (segment (start 135.589977 117.9) (end 135.664477 117.8255) (width 0.15) (layer "B.Cu") (net 3))

Commit message: Add a pull-up register to the CHIP-PU pin.
Signed-off-by: Kazuki Iida <elkel53930@gmail.com>
Parts:
- added R2: 0603 10k, Resistor_SMD:R_0201_0603Metric, F.Cu at (149.5, 121.0)
Routing:
- net /CHIP_PU: track 20.1 -> 26.7 mm
- net +3V0: track 162.3 -> 166.5 mm, vias 15 -> 16
Changed lines of the file:
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@@
     (pad "" np_thru_hole circle (at 0 0) (size 1.4 1.4) (drill 1.4) (layers "*.Cu" "*.Mask"))
+  )
+  (footprint "Resistor_SMD:R_0201_0603Metric" (layer "F.Cu")
+    (at 149.5 121)
+    (descr "Resistor SMD 0201 (0603 Metric), square (rectangular) end terminal, IPC_7351 nominal, (Body size source: https://www.vishay.com/docs/20052/crcw0201e3.pdf), generated with kicad-footprint-generator")
+    (tags "resistor")
+    (property "Sheetfile" "extraice.kicad_sch")
+    (property "Sheetname" "")
+    (property "ki_description" "Resistor")
+    (property "ki_keywords" "R res resistor")
+    (attr smd)
+    (fp_text reference "R2" (at 0 1) (layer "F.SilkS")
+        (effects (font (size 0.6 0.6) (thickness 0.1) bold))
+    )
+    (fp_text value "0603 10k" (at 0 1.05) (layer "F.Fab")
+        (effects (font (size 1 1) (thickness 0.15)))
+    )
+    (fp_text user "${REFERENCE}" (at 0 -0.68) (layer "F.Fab")
+        (effects (font (size 0.25 0.25) (thickness 0.04)))
+    )
+    (fp_line (start -0.7 -0.35) (end 0.7 -0.35)
+      (stroke (width 0.05) (type solid)) (layer "F.CrtYd"))
+    (fp_line (start -0.7 0.35) (end -0.7 -0.35)
+      (stroke (width 0.05) (type solid)) (layer "F.CrtYd"))
+    (fp_line (start 0.7 -0.35) (end 0.7 0.35)
+      (stroke (width 0.05) (type solid)) (layer "F.CrtYd"))
+    (fp_line (start 0.7 0.35) (end -0.7 0.35)
+      (stroke (width 0.05) (type solid)) (layer "F.CrtYd"))
+    (fp_line (start -0.3 -0.15) (end 0.3 -0.15)
+      (stroke (width 0.1) (type solid)) (layer "F.Fab"))
+    (fp_line (start -0.3 0.15) (end -0.3 -0.15)
+      (stroke (width 0.1) (type solid)) (layer "F.Fab"))
+    (fp_line (start 0.3 -0.15) (end 0.3 0.15)
+      (stroke (width 0.1) (type solid)) (layer "F.Fab"))
+    (fp_line (start 0.3 0.15) (end -0.3 0.15)
+      (stroke (width 0.1) (type solid)) (layer "F.Fab"))
+    (pad "" smd roundrect (at -0.345 0) (size 0.318 0.36) (layers "F.Paste") (roundrect_rratio 0.25))
+    (pad "" smd roundrect (at 0.345 0) (size 0.318 0.36) (layers "F.Paste") (roundrect_rratio 0.25))
+    (pad "1" smd roundrect (at -0.32 0) (size 0.46 0.4) (layers "F.Cu" "F.Mask") (roundrect_rratio 0.25)
+      (net 3 "+3V0") (pintype "passive"))
+    (pad "2" smd roundrect (at 0.32 0) (size 0.46 0.4) (layers "F.Cu" "F.Mask") (roundrect_rratio 0.25)
+      (net 60 "/CHIP_PU") (pintype "passive"))
+    (model "${KICAD6_3DMODEL_DIR}/Resistor_SMD.3dshapes/R_0201_0603Metric.wrl"
+      (offset (xyz 0 0 0))
+      (scale (xyz 1 1 1))
+      (rotate (xyz 0 0 0))
+    )
   )
   (footprint "Capacitor_SMD:C_0201_0603Metric" (layer "F.Cu")
@@
   (via (at 130 110) (size 0.5) (drill 0.3) (layers "F.Cu" "B.Cu") (free) (net 1))
   (via (at 145 106) (size 0.5) (drill 0.3) (layers "F.Cu" "B.Cu") (free) (net 1))
-  (via (at 150 121) (size 0.5) (drill 0.3) (layers "F.Cu" "B.Cu") (free) (net 1))
+  (via (at 151 121) (size 0.5) (drill 0.3) (layers "F.Cu" "B.Cu") (free) (net 1))
   (via (at 132.7 91.1) (size 0.5) (drill 0.3) (layers "F.Cu" "B.Cu") (free) (net 1))
   (via (at 152.75 100) (size 0.5) (drill 0.3) (layers "F.Cu" "B.Cu") (free) (net 1))
@@
   (segment (start 144.48 114.2) (end 144.48 114.78) (width 0.15) (layer "F.Cu") (net 3))
   (segment (start 144.2 116.1) (end 144 116.3) (width 0.15) (layer "F.Cu") (net 3))
+  (segment (start 149.18 121) (end 148.5 121) (width 0.15) (layer "F.Cu") (net 3))
   (segment (start 135.7 117.9) (end 135.664477 117.864477) (width 0.15) (layer "F.Cu") (net 3))
   (segment (start 142.5 131.68) (end 142.4455 131.6255) (width 0.15) (layer "F.Cu") (net 3))
@@
   (via (at 130.8 120) (size 0.5) (drill 0.3) (layers "F.Cu" "B.Cu") (net 3))
   (via (at 145.3 116.1) (size 0.5) (drill 0.3) (layers "F.Cu" "B.Cu") (net 3))
+  (via (at 148.5 121) (size 0.5) (drill 0.3) (layers "F.Cu" "B.Cu") (net 3))
   (via (at 144.5 114.8) (size 0.5) (drill 0.3) (layers "F.Cu" "B.Cu") (net 3))
   (via (at 131.4 117.5) (size 0.5) (drill 0.3) (layers "F.Cu" "B.Cu") (net 3))
@@
   (segment (start 144.5 114.8) (end 142.3 114.8) (width 0.3) (layer "B.Cu") (net 3))
   (segment (start 151.351974 91.101974) (end 147.8 91.101974) (width 0.2) (layer "B.Cu") (net 3))
-  (segment (start 144.9505 122.9505) (end 144.9505 119.3495) (width 0.3) (layer "B.Cu") (net 3))
   (segment (start 128.407608 92.898026) (end 128.407608 97.907608) (width 0.2) (layer "B.Cu") (net 3))
   (segment (start 133.4 117.5) (end 131.4 117.5) (width 0.15) (layer "B.Cu") (net 3))
+  (segment (start 148.5 121) (end 144.9505 121) (width 0.15) (layer "B.Cu") (net 3))
   (segment (start 145.3 123.3) (end 144.9505 122.9505) (width 0.3) (layer "B.Cu") (net 3))
   (segment (start 142.3 114.8) (end 136.9 114.8) (width 0.3) (layer "B.Cu") (net 3))
   (segment (start 136.9 114.8) (end 133.8 117.9) (width 0.3) (layer "B.Cu") (net 3))
   (segment (start 147.8 88) (end 144.80659 85.00659) (width 0.2) (layer "B.Cu") (net 3))
+  (segment (start 144.9505 122.9505) (end 144.9505 121) (width 0.3) (layer "B.Cu") (net 3))
   (segment (start 147.8 91.101974) (end 147.8 88) (width 0.2) (layer "B.Cu") (net 3))
+  (segment (start 144.9505 121) (end 144.9505 119.3495) (width 0.3) (layer "B.Cu") (net 3))
   (segment (start 130.8 120) (end 130.8 118.1) (width 0.15) (layer "B.Cu") (net 3))
   (segment (start 142.3 110.2) (end 147.8 104.7) (width 0.3) (layer "B.Cu") (net 3))
@@
   (segment (start 154.875499 119.685499) (end 154.875499 116.275499) (width 0.15) (layer "F.Cu") (net 60))
   (segment (start 141.4 114.647116) (end 141.4 115.05) (width 0.15) (layer "F.Cu") (net 60))
+  (segment (start 150.32 121.5) (end 155.11 121.5) (width 0.15) (layer "F.Cu") (net 60))
   (segment (start 155.9 120.71) (end 154.875499 119.685499) (width 0.15) (layer "F.Cu") (net 60))
   (segment (start 154.875499 116.275499) (end 152.375 113.775) (width 0.15) (layer "F.Cu") (net 60))
+  (segment (start 155.11 121.5) (end 155.9 120.71) (width 0.15) (layer "F.Cu") (net 60))
   (segment (start 142.272116 113.775) (end 141.4 114.647116) (width 0.15) (layer "F.Cu") (net 60))
+  (segment (start 149.82 121) (end 150.32 121.5) (width 0.15) (layer "F.Cu") (net 60))
   (segment (start 152.375 113.775) (end 142.272116 113.775) (width 0.15) (layer "F.Cu") (net 60))
   (segment (start 155.175 118.470305) (end 155.9 119.195305) (width 0.15) (layer "F.Cu") (net 61))

Commit message: Artwork for 4A completed
Need to check details.

Signed-off-by: Kazuki Iida <elkel53930@gmail.com>
Parts:
- removed C14, C15, C16, C5: 0603 50V 0.1uF, Capacitor_SMD:C_0201_0603Metric
- removed R14, R15, R16: 0603 10k, Resistor_SMD:R_0201_0603Metric
- removed SW2: B3U-1000P, Button_Switch_SMD:SW_SPST_B3U-1000P
- removed U4: MB85RC64TA, Library:LCC-8P-M04
- removed X1: 830108208709, Oscillator:Oscillator_SMD_ECS_2520MV-xxx-xx-4Pin_2.5x2.0mm
- added C6: 1608 10V 4.7uF, Capacitor_SMD:C_0603_1608Metric, F.Cu at (131.8, 92.2)
- added D8: 1608 R LED, LED_SMD:LED_0603_1608Metric, F.Cu at (121.0, 109.0)
- added J2: Conn_01x03, Connector_PinHeader_2.00mm:PinHeader_1x03_P2.00mm_Vertical, F.Cu at (148.2, 98.5)
- added R3: 0603 10k, Resistor_SMD:R_0201_0603Metric, F.Cu at (121.0, 111.8)
- C11, C13: value 1005 N/M -> 1608 10V 4.7uF; footprint Capacitor_SMD:C_0402_1005Metric -> Capacitor_SMD:C_0603_1608Metric
- C12: value 0603 50V 0.1uF -> 1608 10V 4.7uF; footprint Capacitor_SMD:C_0201_0603Metric -> Capacitor_SMD:C_0603_1608Metric
- C4: value 3225 25V 22uF -> 1608 10V 4.7uF; footprint Capacitor_SMD:C_1210_3225Metric -> Capacitor_SMD:C_0603_1608Metric
- J1: value Conn_01x02 -> Conn_01x03; footprint Micromouse:B2B-ZH -> Connector_PinHeader_2.00mm:PinHeader_1x03_P2.00mm_Vertical
- R1, R10, R12, R7: value 0603 470 1% -> 1005 470 1%; footprint Resistor_SMD:R_0201_0603Metric -> Resistor_SMD:R_0402_1005Metric
- U7: value ESP32-S3-FN8 -> ESP32-S3-PICO-1-N8R2
- moved C10 45.9 mm to (134.2, 84.2), turned to 180 degrees
- moved U6 43.1 mm to (134.0, 86.8), turned to 0 degrees
- moved G*** 38.6 mm to (129.8, 75.2)
- moved C13 36.4 mm to (131.2, 87.1), turned to 90 degrees
- moved C4 36.0 mm to (131.8, 93.6), turned to 180 degrees
- moved U3 33.6 mm to (130.8, 95.7), turned to 0 degrees
- moved C12 33.4 mm to (131.8, 89.4), turned to 180 degrees
- moved C1 31.2 mm to (126.5, 85.3), turned to -90 degrees
- moved C18 29.4 mm to (148.5, 95.2), turned to -90 degrees
- moved R13 29.3 mm to (129.4, 97.6), turned to 0 degrees
- moved H3 28.6 mm to (126.5, 111.5)
- moved C11 28.2 mm to (131.8, 90.8), turned to 180 degrees
- moved H2 27.7 mm to (153.5, 102.8)
- moved U7 27.5 mm to (140.0, 91.0), turned to -45 degrees
- moved C19 26.9 mm to (141.7, 95.9), turned to 45 degrees
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Connections:
- C11 pad 1: Net-(U7-XTAL_P) -> GND
- C11 pad 2: GND -> +3.3V
- C12 pad 1: +3V0 -> GND
- C12 pad 2: GND -> +3.3V
- C13 pad 1: Net-(U7-XTAL_N) -> GND
- C13 pad 2: GND -> +3.3V
- C21 pad 1: +BATT -> /V_MOT
- C4 pad 1: +3.3V -> GND
- C4 pad 2: GND -> +3.3V
- D5 pad 1: /LED_LEFT_R -> /LED_R
- D6 pad 1: /LED_RIGHT_G -> /LED_G
- D7 pad 1: /LED_FRONT_B -> /LED_B
- J1 pad 1: GND -> Net-(J1-Pin_1)
- J1 pad 2: Net-(J1-Pin_2) -> unconnected-(J1-Pin_2-Pad2)
- SW1 pad 2: Net-(J1-Pin_2) -> +BATT
- SW1 pad 3: +BATT -> /V_MOT
- U10 pad 1: +BATT -> /V_MOT
- U11 pad 1: +BATT -> /V_MOT
- U7 pad 11: /SPI2_MISO -> /SEN_LED_ENA
- U7 pad 12: /SPI2_MOSI -> /LED_SEL0
- U7 pad 13: /SPI2_SCK -> /LED_SEL1
- U7 pad 14: /CS_IMU -> /CS_ENC_L
- U7 pad 15: /CS_ENC_L -> /SPI1_SCK
- U7 pad 16: /SPI1_SCK -> /SPI1_MISO
- U7 pad 17: /SPI1_MISO -> /SPI1_MOSI
- U7 pad 18: /SPI1_MOSI -> /LED_R
- U7 pad 19: /SEN_LED_ENA -> /LED_G
- U7 pad 21: /LED_SEL0 -> /LED_B
- U7 pad 22: /LED_SEL1 -> /SPI2_MISO
- U7 pad 23: /SCL -> unconnected-(U7-GPIO17-Pad23)
- U7 pad 24: /SDA -> unconnected-(U7-GPIO18-Pad24)
- U7 pad 25: /LED_RIGHT_G -> /SPI2_MOSI
- U7 pad 26: /LED_FRONT_B -> /SPI2_SCK
- U7 pad 27: /LED_LEFT_R -> /CS_IMU
- U7 pad 44: Net-(U7-MTCK) -> unconnected-(U7-MTCK-Pad44)
- U7 pad 53: Net-(U7-XTAL_N) -> unconnected-(U7-XTAL_N-Pad53)
- U7 pad 54: Net-(U7-XTAL_P) -> unconnected-(U7-XTAL_P-Pad54)
- U7 pad 6: /SEN_LS -> /SEN_RS
- U7 pad 7: /SEN_LF -> /SEN_RF
- U7 pad 8: /SEN_RF -> /SEN_LF
- U7 pad 9: /SEN_RS -> /SEN_LS
- U9 pad 1: +BATT -> /V_MOT
Routing:
- net /V_MOT: track 0.00 -> 71.4 mm, vias 0 -> 5
- net /SEN_LS: track 75.9 -> 13.4 mm, vias 1 -> 0
- net /SEN_LF: track 63.5 -> 10.4 mm, vias 1 -> 0
- net +3.3V: track 119.4 -> 68.3 mm, vias 2 -> 4
- net /SEN_RF: track 45.7 -> 12.1 mm, vias 1 -> 0
- net /LED_R: track 0.00 -> 31.5 mm
- net /LED_LEFT_R: track 30.8 -> 0.00 mm, vias 2 -> 0
- net /LED_G: track 0.00 -> 30.7 mm
- net /SEN_LED_ENA: track 42.9 -> 13.1 mm
- net /LED_B: track 0.00 -> 29.5 mm
- net /PWM_V: track 3.99 -> 32.5 mm
- net /LED_FRONT_B: track 28.0 -> 0.00 mm, vias 2 -> 0
- net /TXD: track 14.6 -> 42.3 mm
- net /GPIO0: track 19.8 -> 47.4 mm
- net /LED_SEL1: track 46.0 -> 18.4 mm
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Other:
- board size 77 x 57.8 mm -> 77 x 68.5 mm
- board text added: "ExtraICE-4A 2024"
- board text removed: "A:Mac ExtraICE-4 2023"
- board text removed: "ExtraICE-4 2023"

Commit message: EXTRAICE5
Parts:
- removed C18, C21: 2012 35V 10uF, Capacitor_SMD:C_0805_2012Metric
- removed C19: 0603 50V 0.1uF, Capacitor_SMD:C_0201_0603Metric
- removed Q2, Q3, Q4: L-31ROPT1C, Micromouse:OSI5FU3A11C
- added BT1: 100mAh LiPo, Micromouse:Battery, B.Cu at (170.9, 87.2)
- added C14: 1005 50V 0.1uF, Capacitor_SMD:C_0402_1005Metric, F.Cu at (99.0, 93.3)
- added C15: 1005 50V 0.1uF, Capacitor_SMD:C_0402_1005Metric, F.Cu at (141.2, 97.6)
- added C16: 1005 50V 0.1uF, Capacitor_SMD:C_0402_1005Metric, F.Cu at (139.2, 97.6)
- added C17: 2012 35V 10uF, Capacitor_SMD:C_0805_2012Metric, F.Cu at (170.9, 104.9)
- added C5: 4532 10u 16V, Capacitor_SMD:C_1812_4532Metric, F.Cu at (143.5, 123.5)
- added H5: Φ2.2, MountingHole:MountingHole_2.2mm_M2, F.Cu at (96.5, 90.0)
- added H6: Φ2.2, MountingHole:MountingHole_2.2mm_M2, F.Cu at (87.5, 90.0)
- added J11: Conn_01x03, Connector_PinSocket_2.00mm:PinSocket_1x03_P2.00mm_Vertical, B.Cu at (179.1, 89.0)
- added J12: Conn_01x02, Micromouse:B2B-ZH, F.Cu at (175.3, 106.6)
- added LS1: SMT-0440-T-2-R, Library:SMT-0440-T-2-R, F.Cu at (156.8, 113.8)
- added R14: 1005 10k, Resistor_SMD:R_0402_1005Metric, F.Cu at (155.3, 117.3)
- added R15: 1005 1k, Resistor_SMD:R_0402_1005Metric, F.Cu at (142.6, 96.4)
- added R16: 1005 1k, Resistor_SMD:R_0402_1005Metric, F.Cu at (142.6, 95.4)
- added R17: 1005 1k, Resistor_SMD:R_0402_1005Metric, F.Cu at (124.5, 111.4)
- added R18: 1005 1k, Resistor_SMD:R_0402_1005Metric, F.Cu at (121.8, 113.2)
- added R19: 1005 6.2, Resistor_SMD:R_0402_1005Metric, B.Cu at (135.5, 89.5)
- added R20: 1005 10k, Resistor_SMD:R_0402_1005Metric, F.Cu at (170.9, 102.8)
- added R21: 1005 1k, Resistor_SMD:R_0402_1005Metric, F.Cu at (170.9, 96.9)
- added U13: ~, Micromouse:PhotoSensorL, F.Cu at (135.1, 72.5)
- added U14: ~, Micromouse:PhotoSensorR, F.Cu at (144.9, 72.5)
- added U15: ~, Micromouse:PhotoSensorR, F.Cu at (155.5, 87.4)
- added U16: LTC4054ES5-4.2, Package_TO_SOT_SMD:TSOT-23-5, F.Cu at (170.9, 100.1)
- added U4: TLA2528IRTER, Package_DFN_QFN:WQFN-16-1EP_3x3mm_P0.5mm_EP1.68x1.68mm, F.Cu at (142.5, 84.5)
- C1: value 1608 35V 1uF -> 1608 10V 4.7uF
- C10: value 1608 35V 1uF -> 1005 50V 0.1uF; footprint Capacitor_SMD:C_0603_1608Metric -> Capacitor_SMD:C_0402_1005Metric
- C11, C13: value 1608 10V 4.7uF -> 1005 50V 0.1uF; footprint Capacitor_SMD:C_0603_1608Metric -> Capacitor_SMD:C_0402_1005Metric
- C12: value 1608 10V 4.7uF -> 1608 35V 1uF
- C2: value 2012 35V 10uF -> 1608 10V 4.7uF; footprint Capacitor_SMD:C_0805_2012Metric -> Capacitor_SMD:C_0603_1608Metric
- C3: value 0603 50V 0.1uF -> 1608 10V 4.7uF; footprint Capacitor_SMD:C_0201_0603Metric -> Capacitor_SMD:C_0603_1608Metric
- C4: value 1608 10V 4.7uF -> 4532 10u 16V; footprint Capacitor_SMD:C_0603_1608Metric -> Capacitor_SMD:C_1812_4532Metric
- C6: value 1608 10V 4.7uF -> 2012 35V 10uF; footprint Capacitor_SMD:C_0603_1608Metric -> Capacitor_SMD:C_0805_2012Metric
- C7: value 0603 50V 0.1uF -> 1005 50V 0.1uF; footprint Capacitor_SMD:C_0201_0603Metric -> Capacitor_SMD:C_0402_1005Metric
- C8: value 0603 50V 0.1uF -> 4532 10u 16V; footprint Capacitor_SMD:C_0201_0603Metric -> Capacitor_SMD:C_1812_4532Metric
- C9: value 0603 50V 0.1uF -> 1608 35V 1uF; footprint Capacitor_SMD:C_0201_0603Metric -> Capacitor_SMD:C_0603_1608Metric
- D1, D2: value OSI5FU3A11C -> 1608 LED; footprint Micromouse:OSI5FU3A11C -> LED_SMD:LED_0603_1608Metric
- D3: value OSI5FU3A11C -> BAS516; footprint Micromouse:OSI5FU3A11C -> Diode_SMD:D_SOD-523
- D4: value OSI5FU3A11C -> 1608 R LED; footprint Micromouse:OSI5FU3A11C -> LED_SMD:LED_0603_1608Metric
- D5, D8: value 1608 R LED -> 1608 LED
- D6: value 1608 G LED -> 1608 LED
- D7: value 1608 B LED -> 1608 LED
- J10: value Conn_01x02 -> Conn_01x03; footprint Micromouse:MotorPad -> Connector_PinSocket_2.00mm:PinSocket_1x03_P2.00mm_Vertical; moved to B.Cu
- J3: value EncSide -> Conn_01x05; footprint Micromouse:EncoderTerminal -> Connector_PinHeader_1.27mm:PinHeader_1x05_P1.27mm_Vertical
- J4: value MainSide -> Conn_01x02; footprint Micromouse:EncoderTerminal -> Connector_PinHeader_1.27mm:PinHeader_1x02_P1.27mm_Vertical
- J5: value Conn_01x05 -> Conn_01x02; footprint Connector_PinHeader_1.27mm:PinHeader_1x05_P1.27mm_Vertical -> Connector_PinHeader_1.27mm:PinHeader_1x02_P1.27mm_Vertical
- J8: value Conn_01x02 -> EncSide; footprint Micromouse:MotorPad -> Micromouse:EncoderTerminal
- J9: value Conn_01x02 -> MainSide; footprint Micromouse:MotorPad -> Micromouse:EncoderTerminal
- Q1: value L-31ROPT1C -> MMBT3904; footprint Micromouse:OSI5FU3A11C -> Package_TO_SOT_SMD:SOT-23
- R1: value 1005 470 1% -> 1005 1k
- R10, R12: moved to B.Cu
- R11: value 0603 6.2 -> 1005 470 1%; footprint Resistor_SMD:R_0201_0603Metric -> Resistor_SMD:R_0402_1005Metric; moved to B.Cu
- R13: value 0603 22k -> 1005 470 1%; footprint Resistor_SMD:R_0201_0603Metric -> Resistor_SMD:R_0402_1005Metric; moved to B.Cu
- R2, R3: value 0603 10k -> 1005 10k; footprint Resistor_SMD:R_0201_0603Metric -> Resistor_SMD:R_0402_1005Metric
- R4, R6, R9: value 0603 1k -> 1005 1k; footprint Resistor_SMD:R_0201_0603Metric -> Resistor_SMD:R_0402_1005Metric
- R5: value 0603 1k -> 1005 10k; footprint Resistor_SMD:R_0201_0603Metric -> Resistor_SMD:R_0402_1005Metric
- R8: value 0603 10k -> 1005 1k; footprint Resistor_SMD:R_0201_0603Metric -> Resistor_SMD:R_0402_1005Metric
- U1: value DG2034EDN -> XC6221B302GR; footprint Library:QFN-12-1EP_3x3mm_P0.5_EP1.15x1.15 -> Package_TO_SOT_SMD:SOT-23-5
- U10: value DRV8837C -> DG2034EDN; footprint Package_SON:WSON-8-1EP_2x2mm_P0.5mm_EP0.9x1.6mm -> Library:QFN-12-1EP_3x3mm_P0.5_EP1.15x1.15
- U11: value DRV8837C -> BCR421; footprint Package_SON:WSON-8-1EP_2x2mm_P0.5mm_EP0.9x1.6mm -> Library:SOT-26
- U12: value AS5047D -> ~; footprint Package_SO:TSSOP-14_4.4x5mm_P0.65mm -> Micromouse:PhotoSensorL
- U2: value BCR421 -> DRV8837C; footprint Library:SOT-26 -> Package_SON:WSON-8-1EP_2x2mm_P0.5mm_EP0.9x1.6mm
- U3: value MUN12AD01-SG -> ESP32-S3-PICO-1-N8R2; footprint Library:MUN12AD01-SG -> Package_DFN_QFN:QFN-56-1EP_7x7mm_P0.4mm_EP4x4mm
- U5: value LSM6DSR -> DRV8837C; footprint Package_LGA:Bosch_LGA-14_3x2.5mm_P0.5mm -> Package_SON:WSON-8-1EP_2x2mm_P0.5mm_EP0.9x1.6mm
- U6: value XC6221B302GR -> MB85RC64TA; footprint Package_TO_SOT_SMD:SOT-23-5 -> Library:LCC-8P-M04
- U7: value ESP32-S3-PICO-1-N8R2 -> AS5047D; footprint Package_DFN_QFN:QFN-56-1EP_7x7mm_P0.4mm_EP4x4mm -> Package_SO:TSSOP-14_4.4x5mm_P0.65mm
- U9: value DRV8837C -> LSM6DSR; footprint Package_SON:WSON-8-1EP_2x2mm_P0.5mm_EP0.9x1.6mm -> Package_LGA:Bosch_LGA-14_3x2.5mm_P0.5mm
- moved J3 77.0 mm to (153.2, 118.8), turned to 180 degrees
- moved J8 58.1 mm to (96.5, 94.5), turned to 180 degrees
- moved U7 52.5 mm to (87.5, 90.0), turned to 0 degrees
- moved D8 52.1 mm to (170.9, 94.1), turned to 90 degrees
- moved U2 45.8 mm to (147.0, 122.0)
- moved D4 43.8 mm to (123.5, 117.0)
- moved C13 41.7 mm to (90.0, 93.5), turned to 180 degrees
- moved U10 40.2 mm to (135.5, 81.5)
- moved U11 39.1 mm to (135.5, 86.6), turned to -90 degrees
- moved C8 37.1 mm to (136.0, 123.5), turned to -90 degrees
- moved J10 37.1 mm to (162.7, 89.0), turned to 180 degrees
- moved R7 35.9 mm to (153.3, 111.8), turned to 0 degrees
- moved D3 35.7 mm to (157.5, 110.8), turned to 180 degrees
- moved R5 35.6 mm to (146.1, 92.1)
- moved D2 35.5 mm to (134.0, 113.2), turned to 180 degrees
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Connections:
- C1 pad 1: +3.3V -> GND
- C1 pad 2: GND -> +BATT
- C10 pad 1: +3V0 -> Net-(U3-VDD_SPI)
- C11 pad 1: GND -> +3V0
- C11 pad 2: +3.3V -> GND
- C12 pad 1: GND -> +BATT
- C12 pad 2: +3.3V -> GND
- C13 pad 1: GND -> Net-(J6-Pin_1)
- C13 pad 2: +3.3V -> Net-(J6-Pin_6)
- C3 pad 2: +3V0 -> +BATT
- C4 pad 1: GND -> +3V0
- C4 pad 2: +3.3V -> GND
- C6 pad 1: GND -> +3V0
- C6 pad 2: +3.3V -> GND
- C7 pad 1: GND -> +3V0
- C7 pad 2: +3V0 -> GND
- C8 pad 1: GND -> /V_MOT
- C8 pad 2: +3V0 -> GND
- C9 pad 1: +3V0 -> GND
- C9 pad 2: GND -> Net-(U4-DECAP)
- D1 pad 2: +3.3V -> +3V0
- D2 pad 2: +3.3V -> +3V0
- D3 pad 1: Net-(D3-K) -> +3V0
- D3 pad 2: +3.3V -> Net-(D3-A)
- D4 pad 1: Net-(D4-K) -> GND
- D4 pad 2: +3.3V -> Net-(D4-A)
- D5 pad 1: /LED_R -> Net-(D5-K)
- D5 pad 2: Net-(D5-A) -> +3V0
- D6 pad 1: /LED_G -> Net-(D6-K)
- D6 pad 2: Net-(D6-A) -> +3V0
- D7 pad 1: /LED_B -> Net-(D7-K)
- D7 pad 2: Net-(D7-A) -> +3V0
- D8 pad 1: GND -> Net-(D8-K)
- J1 pad 1: Net-(J1-Pin_1) -> /V_MOT
- J1 pad 2: unconnected-(J1-Pin_2-Pad2) -> /V_MOT
- J10 pad 1: Net-(J10-Pin_1) -> Net-(BT1-+)
- J10 pad 2: Net-(J10-Pin_2) -> Net-(BT1-+)
- J2 pad 2: unconnected-(J2-Pin_2-Pad2) -> GND
- J2 pad 3: Net-(J1-Pin_1) -> GND
- J3 pad 1: Net-(J3-Pin_1) -> /TXD
- J3 pad 2: Net-(J3-Pin_2) -> /RXD
- J3 pad 3: Net-(J3-Pin_3) -> /CHIP_PU
- J3 pad 4: Net-(J3-Pin_4) -> /GPIO0
- J3 pad 5: Net-(J3-Pin_5) -> GND
- J4 pad 1: +3V0 -> Net-(J4-Pin_1)
- J4 pad 2: /SPI1_MOSI -> Net-(J4-Pin_2)
- J5 pad 1: /TXD -> Net-(J5-Pin_1)
- J5 pad 2: /RXD -> Net-(J5-Pin_2)
- J7 pad 5: /CS_ENC_L -> /CS_ENC_R
- J9 pad 1: Net-(J9-Pin_1) -> +3V0
- J9 pad 2: Net-(J9-Pin_2) -> /SPI1_MOSI
- Q1 pad 1: +3V0 -> Net-(Q1-B)
- Q1 pad 2: /SEN_LS -> GND
- R1 pad 1: /SEN_LS -> Net-(D1-K)
- R1 pad 2: GND -> /LED_0
- R10 pad 1: /SEN_RF -> /SEN_LF
- R11 pad 1: Net-(U2-Rext) -> /SEN_LS
- R13 pad 1: GND -> /SEN_RF
- R13 pad 2: Net-(U3-FB) -> GND
- R2 pad 1: +3V0 -> Net-(D4-A)
- R2 pad 2: /CHIP_PU -> +BATT
- R3 pad 1: Net-(D8-A) -> /BATT_SEN
- R4 pad 1: +3V0 -> Net-(D2-K)
- R4 pad 2: Net-(D5-A) -> /LED_1
- R5 pad 1: +3V0 -> GND
- R5 pad 2: Net-(D6-A) -> /BATT_SEN
- R6 pad 1: +3V0 -> Net-(D5-K)
- R6 pad 2: Net-(D7-A) -> /LED_2
- R7 pad 1: /SEN_LF -> /BUZZ
- R7 pad 2: GND -> Net-(Q1-B)
- R8 pad 1: /BATT_SEN -> Net-(D6-K)
- R8 pad 2: +BATT -> /LED_3
- R9 pad 1: GND -> Net-(D7-K)
- R9 pad 2: /BATT_SEN -> /LED_4
- U1 pad 1: Net-(D4-K) -> +BATT
- U1 pad 3: Net-(D3-K) -> +BATT
- U1 pad 4: +3.3V -> unconnected-(U1-NC-Pad4)
- U1 pad 5: unconnected-(U1-NC-Pad5) -> +3V0
- U10 pad 1: /V_MOT -> Net-(U10-S1)
- U10 pad 2: Net-(J9-Pin_1) -> GND
- U10 pad 3: Net-(J9-Pin_2) -> Net-(U10-S3)
- U10 pad 4: GND -> +BATT
- U10 pad 5: /CWCCW_L -> unconnected-(U10-NC-Pad5)
- U10 pad 6: /PWM_L -> +BATT
- U10 pad 7: /MOT_SLEEP -> Net-(U10-S4)
- U10 pad 8: +3V0 -> Net-(U10-COM)
- U10 pad 9: GND -> Net-(U10-S2)
- U11 pad 1: /V_MOT -> /SEN_LED_ENA
- U11 pad 2: Net-(J10-Pin_1) -> Net-(U10-COM)
- U11 pad 3: Net-(J10-Pin_2) -> Net-(U10-COM)
- U11 pad 5: GND -> Net-(U10-COM)
- U11 pad 6: /PWM_V -> Net-(U11-Rext)
- U12 pad 1: Net-(J6-Pin_5) -> /SEN_LF
- U12 pad 2: Net-(J6-Pin_4) -> +3V0
- U12 pad 3: Net-(J6-Pin_3) -> +BATT
- U12 pad 4: Net-(J6-Pin_2) -> Net-(U10-S2)
- U2 pad 1: /SEN_LED_ENA -> /V_MOT
- U2 pad 2: Net-(U1-COM) -> Net-(J4-Pin_1)
- U2 pad 3: Net-(U1-COM) -> Net-(J4-Pin_2)
- U2 pad 5: Net-(U1-COM) -> /CWCCW_R
- U2 pad 6: Net-(U2-Rext) -> /PWM_R
- U3 pad 2: GND -> +3V0
- U3 pad 3: Net-(U3-FB) -> +3V0
- U3 pad 4: +BATT -> /CHIP_PU
- U3 pad 5: +BATT -> /GPIO0
- U3 pad 6: +3.3V -> unconnected-(U3-GPIO1-Pad6)
- U5 pad 1: /SPI2_MISO -> /V_MOT
- U5 pad 2: GND -> Net-(J5-Pin_1)
- U5 pad 3: GND -> Net-(J5-Pin_2)
- U5 pad 4: unconnected-(U5-INT1-Pad4) -> GND
- U5 pad 5: +3V0 -> /CWCCW_L
- U5 pad 6: GND -> /PWM_L
- U5 pad 7: GND -> /MOT_SLEEP
- U5 pad 8: +3V0 -> /V_MOT
- U5 pad 9: unconnected-(U5-INT2-Pad9) -> GND
- U6 pad 1: +3.3V -> GND
- U6 pad 3: +3.3V -> GND
- U6 pad 4: unconnected-(U6-NC-Pad4) -> GND
- U6 pad 5: +3V0 -> /SCL1
- U7 pad 1: unconnected-(U7-LNA_IN-Pad1) -> Net-(J6-Pin_5)
- U7 pad 10: /BATT_SEN -> unconnected-(U7-U-Pad10)
- U7 pad 11: /SEN_LED_ENA -> unconnected-(U7-VDD-Pad11)
- U7 pad 12: /LED_SEL0 -> Net-(J6-Pin_1)
- U7 pad 13: /LED_SEL1 -> Net-(J6-Pin_6)
- U7 pad 14: /CS_ENC_L -> unconnected-(U7-I/PWM-Pad14)
- U7 pad 2: +3V0 -> Net-(J6-Pin_4)
- U7 pad 3: +3V0 -> Net-(J6-Pin_3)
- U7 pad 4: /CHIP_PU -> Net-(J6-Pin_2)
- U7 pad 5: /GPIO0 -> Net-(J6-Pin_6)
- U7 pad 6: /SEN_RS -> unconnected-(U7-B-Pad6)
- U7 pad 7: /SEN_RF -> unconnected-(U7-A-Pad7)
- U7 pad 8: /SEN_LF -> unconnected-(U7-W/PWM-Pad8)
- U7 pad 9: /SEN_LS -> unconnected-(U7-V-Pad9)
- U8 pad 1: Net-(J3-Pin_5) -> Net-(J8-Pin_5)
- U8 pad 12: Net-(J3-Pin_1) -> Net-(J8-Pin_1)
- U8 pad 13: Net-(J3-Pin_6) -> Net-(J8-Pin_6)
- U8 pad 2: Net-(J3-Pin_4) -> Net-(J8-Pin_4)
- U8 pad 3: Net-(J3-Pin_3) -> Net-(J8-Pin_3)
- U8 pad 4: Net-(J3-Pin_2) -> Net-(J8-Pin_2)
- U8 pad 5: Net-(J3-Pin_6) -> Net-(J8-Pin_6)
- U9 pad 1: /V_MOT -> /SPI2_MISO
- U9 pad 2: Net-(J8-Pin_1) -> GND
- U9 pad 3: Net-(J8-Pin_2) -> GND
- U9 pad 4: GND -> unconnected-(U9-INT1-Pad4)
- U9 pad 5: /CWCCW_R -> +3V0
- U9 pad 6: /PWM_R -> GND
- U9 pad 7: /MOT_SLEEP -> GND
- U9 pad 9: GND -> unconnected-(U9-INT2-Pad9)
Routing:
- net +BATT: track 37.8 -> 131.8 mm, vias 2 -> 9
- net +3V0: track 161.2 -> 242.6 mm, vias 13 -> 19
- net +3.3V: track 68.3 -> 0.00 mm, vias 4 -> 0
- net GND: track 9.85 -> 74.4 mm, vias 74 -> 98
- net Net-(BT1--): track 0.00 -> 43.9 mm, vias 0 -> 1
- net /GPIO0: track 47.4 -> 10.4 mm
- net /CHIP_PU: track 49.7 -> 13.0 mm
- net /RXD: track 41.7 -> 5.38 mm
- net /TXD: track 42.3 -> 6.35 mm
- net /PWM_V: track 32.5 -> 0.00 mm
- net /LED_R: track 31.5 -> 0.00 mm
- net /LED_G: track 30.7 -> 0.00 mm
- net /SDA0: track 0.00 -> 30.3 mm, vias 0 -> 2
- net /LED_B: track 29.5 -> 0.00 mm
- net /SCL0: track 0.00 -> 27.5 mm
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- added copper zone on F.Cu, net Net-(BT1-+)
- added copper zone on B.Cu, net Net-(BT1--)
Other:
- board size 77 x 68.5 mm -> 96.8 x 61 mm
- board text added: "E"
- board text added: "EXTRAICE5"
- board text added: "G"
- board text added: "PU"
- board text added: "R"
- board text added: "T"
- board text removed: "ExtraICE-4A 2024"
